File: eagle/freiBot.brd (EAGLE design)
At the start: 100 x 80 mm, 13 parts, among them IC1 L293D

Commit message: new eagle schematic
Parts:
- added ARDUINO_LED, BUTTON, NEOPIXEL, SCL, SDA, WHISKER: (no value), pinhead:1X01
- added C4: (no value), rcl:E5-8,5
- added C5: 100n, rcl:C050-025X075
- added IR-LED: (no value), 0-svo:LED5MM
- added IR1: (no value), 0-svo:SFH511*
- added R4: 270, rcl:0309/12
- added R5: 100, rcl:0309/10
- moved RIGHTMOTOR1 13.7 mm to (20.3, 20.3)
- moved RIGHTMOTOR2 11.4 mm to (27.9, 20.3)
- moved RIGHTLED 10.2 mm to (69.8, 73.7), turned to 0 degrees
- moved R1 8.98 mm to (71.1, 52.1), turned to 90 degrees
- moved G1 7.18 mm to (30.5, 10.2)
- moved IC1 5.68 mm to (24.1, 36.8)
- moved LEFTMOTOR1 5.68 mm to (27.9, 55.9)
- moved C2 5.68 mm to (19.1, 45.7)
- moved LEFTMOTOR2 5.68 mm to (20.3, 55.9)
- moved C1 5.08 mm to (29.2, 25.4)
- moved LEFTLED 5.08 mm to (26.7, 73.7)
- moved U$1 5.08 mm to (40.6, 25.4)
- moved R2 4.02 mm to (68.6, 52.1), turned to 90 degrees
Connections:
- new net +5V: C2.1, IC1.16, R5.2, U$1.+5V
- new net N$17: SDA.1, U$1.A4
- new net N$18: SCL.1, U$1.A5
- new net N$19: ARDUINO_LED.1, U$1.D13
- new net N$20: U$1.D12, WHISKER.1
- new net N$21: BUTTON.1, U$1.D11
- new net N$22: NEOPIXEL.1, U$1.D7
- new net N$23: IR1.1, U$1.D4
- new net N$24: R4.1, U$1.D5
- new net VCC: C4.+, C5.1, IR1.3, R5.1
- net GND: now also C4.-, C5.2, IR-LED.K, IR1.2
- net N$12: now also IR-LED.A, R4.2; no longer C2.1, IC1.16, U$1.+5V
Routing:
- net N$23: track 0.00 -> 124.5 mm, vias 0 -> 4
- net +5V: track 0.00 -> 73.7 mm, vias 0 -> 2
- net GND: track 189.0 -> 231.1 mm, vias 6 -> 9
- net N$12: track 63.5 -> 101.6 mm, vias 2 -> 4
- net VCC: track 0.00 -> 20.3 mm, vias 0 -> 2
- net N$3: track 81.3 -> 63.5 mm
- net N$16: track 43.2 -> 58.4 mm
- net N$13: track 20.3 -> 5.08 mm
- net N$24: track 0.00 -> 12.7 mm
- net N$2: track 58.4 -> 45.7 mm
- net N$11: track 50.8 -> 63.5 mm, vias 2 -> 4
- net N$14: track 15.2 -> 5.08 mm
- net N$4: track 22.9 -> 12.7 mm
- net N$8: track 20.3 -> 12.7 mm
- net N$5: track 63.5 -> 55.9 mm
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
Commit message: bluetooth modul hc05 connection added
Parts:
- added BLUETOOTH_HC05: (no value), pinhead:1X06
Connections:
- new net BLUE_KEY: BLUETOOTH_HC05.5
- new net BLUE_LED: BLUETOOTH_HC05.6
- new net BLUE_RXD_ARDUINO_TXD: BLUETOOTH_HC05.4, U$1.D8
- new net BLUE_TXD_ARDUINO_RXD: BLUETOOTH_HC05.3, U$1.D6
- net +5V: now also BLUETOOTH_HC05.1
- net GND: now also BLUETOOTH_HC05.2
Routing:
- net +5V: track 73.7 -> 149.9 mm, vias 2 -> 6
- net BLUE_RXD_ARDUINO_TXD: track 0.00 -> 48.3 mm, vias 0 -> 2
- net BLUE_TXD_ARDUINO_RXD: track 0.00 -> 35.6 mm, vias 0 -> 2
- net GND: track 231.1 -> 238.8 mm
Changed lines of the file:
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@@
 </element>
 <element name="RIGHTMOTOR2" library="pinhead" package="1X01" value="" x="27.94" y="20.32" smashed="yes">
-<attribute name="NAME" x="29.1338" y="17.0688" size="1.27" layer="25" ratio="10"/>
+<attribute name="NAME" x="26.5938" y="17.0688" size="1.27" layer="25" ratio="10"/>
 <attribute name="VALUE" x="26.67" y="17.145" size="1.27" layer="27"/>
 </element>
@@
 <element name="C5" library="rcl" package="C050-025X075" value="100n" x="43.18" y="71.12"/>
 <element name="R5" library="rcl" package="0309/10" value="100" x="45.72" y="66.04"/>
+<element name="BLUETOOTH_HC05" library="pinhead" package="1X06" value="" x="46.99" y="15.24" rot="R180"/>
 </elements>
 <signals>
@@
 <via x="55.88" y="68.58" extent="1-16" drill="0.6" shape="square"/>
 <wire x1="55.88" y1="68.58" x2="55.88" y2="55.88" width="1.27" layer="16"/>
+<contactref element="BLUETOOTH_HC05" pad="2"/>
+<wire x1="50.8" y1="15.24" x2="50.8" y2="22.86" width="1.27" layer="16"/>
 </signal>
 <signal name="N$5">
@@
 <contactref element="IC1" pad="16"/>
 <contactref element="U$1" pad="+5V"/>
-<wire x1="15.24" y1="40.64" x2="15.24" y2="45.72" width="1.27" layer="16"/>
+<wire x1="15.24" y1="43.18" x2="15.24" y2="45.72" width="1.27" layer="16"/>
 <wire x1="15.24" y1="45.72" x2="15.24" y2="53.34" width="1.27" layer="16"/>
 <via x="15.24" y="53.34" extent="1-16" drill="0.6" shape="square"/>
@@
 <contactref element="R5" pad="2"/>
 <wire x1="50.8" y1="53.34" x2="50.8" y2="66.04" width="1.27" layer="16"/>
+<contactref element="BLUETOOTH_HC05" pad="1"/>
+<wire x1="53.34" y1="15.24" x2="53.34" y2="12.7" width="1.27" layer="16"/>
+<via x="53.34" y="12.7" extent="1-16" drill="0.6" shape="square"/>
+<wire x1="53.34" y1="12.7" x2="12.7" y2="12.7" width="1.27" layer="1"/>
+<via x="12.7" y="12.7" extent="1-16" drill="0.6" shape="square"/>
+<wire x1="12.7" y1="12.7" x2="12.7" y2="43.18" width="1.27" layer="16"/>
+<via x="12.7" y="43.18" extent="1-16" drill="0.6" shape="square"/>
+<wire x1="12.7" y1="43.18" x2="15.24" y2="43.18" width="1.27" layer="1"/>
+<via x="15.24" y="43.18" extent="1-16" drill="0.6" shape="square"/>
+<wire x1="15.24" y1="43.18" x2="15.24" y2="40.64" width="1.27" layer="16"/>
 </signal>
 <signal name="VCC">
@@
 <wire x1="58.42" y1="71.12" x2="58.42" y2="73.66" width="1.27" layer="16"/>
 </signal>
+<signal name="BLUE_KEY">
+<contactref element="BLUETOOTH_HC05" pad="5"/>
+</signal>
+<signal name="BLUE_LED">
+<contactref element="BLUETOOTH_HC05" pad="6"/>
+</signal>
+<signal name="BLUE_TXD_ARDUINO_RXD">
+<contactref element="BLUETOOTH_HC05" pad="3"/>
+<contactref element="U$1" pad="D6"/>
+<via x="48.26" y="10.16" extent="1-16" drill="0.6" shape="square"/>
+<wire x1="48.26" y1="10.16" x2="63.5" y2="10.16" width="1.27" layer="1"/>
+<via x="63.5" y="10.16" extent="1-16" drill="0.6" shape="square"/>
+<wire x1="63.5" y1="10.16" x2="63.5" y2="25.4" width="1.27" layer="16"/>
+<wire x1="48.26" y1="10.16" x2="48.26" y2="15.24" width="1.27" layer="16"/>
+</signal>
+<signal name="BLUE_RXD_ARDUINO_TXD">
+<contactref element="BLUETOOTH_HC05" pad="4"/>
+<contactref element="U$1" pad="D8"/>
+<via x="45.72" y="7.62" extent="1-16" drill="0.6" shape="square"/>
+<wire x1="45.72" y1="7.62" x2="68.58" y2="7.62" width="1.27" layer="1"/>
+<via x="68.58" y="7.62" extent="1-16" drill="0.6" shape="square"/>
+<wire x1="68.58" y1="7.62" x2="68.58" y2="25.4" width="1.27" layer="16"/>
+<wire x1="45.72" y1="7.62" x2="45.72" y2="15.24" width="1.27" layer="16"/>
+</signal>
 </signals>

Commit message: additional pins in schematic added
Parts:
- added 3V3, A6, A7, AREF, RESET, RX, TX: (no value), pinhead:1X01
- added A1: V5V, pinhead:1X01
- added A2: VGND, pinhead:1X01
- moved BLUETOOTH_HC05 11.4 mm to (36.8, 10.2)
- moved LEFTMOTOR1 11.4 mm to (17.8, 50.8)
- moved LEFTMOTOR2 11.4 mm to (10.2, 50.8)
- moved R1 11.4 mm to (61.0, 47.0)
- moved SCL 11.4 mm to (48.3, 38.1)
- moved SDA 11.4 mm to (50.8, 38.1)
- moved G1 11.4 mm to (20.3, 5.08)
- moved RIGHTMOTOR1 11.4 mm to (10.2, 15.2)
- moved RIGHTMOTOR2 11.4 mm to (17.8, 15.2)
- moved R5 11.4 mm to (35.6, 61.0)
- moved C1 11.4 mm to (19.1, 20.3)
- moved C2 11.4 mm to (8.89, 40.6)
- moved IC1 11.4 mm to (14.0, 31.8)
- moved LEFTLED 11.4 mm to (16.5, 68.6)
- moved U$1 11.4 mm to (30.5, 20.3)
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Connections:
- new net N$25: A6.1, U$1.A6
- new net N$26: 3V3.1, U$1.3V3
- new net N$27: AREF.1, U$1.AREF
- new net N$28: A7.1, U$1.A7
- new net N$29: RESET.1, U$1.RESET
- new net N$30: TX.1, U$1.D1/TX
- new net N$31: RX.1, U$1.D0/RX
- net +5V: now also A1.1
- net GND: now also A2.1
Routing:
- net +5V: track 149.9 -> 154.9 mm
- net N$25: track 0.00 -> 5.08 mm
- net N$23: track 124.5 -> 119.4 mm
- net GND: track 238.8 -> 241.3 mm
- net N$31: track 0.00 -> 2.54 mm
- net N$30: track 0.00 -> 2.54 mm
- net N$29: track 0.00 -> 2.54 mm
- net N$28: track 0.00 -> 2.54 mm
- net N$27: track 0.00 -> 2.54 mm
- net N$26: track 0.00 -> 2.54 mm
- net N$24: track 12.7 -> 10.2 mm
- net N$22: track 5.08 -> 2.54 mm
- net N$21: track 5.08 -> 2.54 mm
- net N$20: track 5.08 -> 2.54 mm
- net N$12: track 101.6 -> 99.1 mm
Other:
- board size 100 x 80 mm -> 79.7 x 72.4 mm
