File: eagle/freiBot.sch (EAGLE design)
At the start: 13 parts, among them IC1 L293D

Commit message: new eagle schematic
Parts:
- added ARDUINO_LED, BUTTON, NEOPIXEL, SCL, SDA, WHISKER: (no value), pinhead:PINHD-1X1
- added C4: (no value), rcl:CPOL-EUE5-8.5
- added C5: 100n, rcl:C-EU050-025X075
- added IR-LED: (no value), 0-svo:LED5MM
- added IR1: (no value), 0-svo:SFH5110
- added R4: 270, rcl:R-EU_0309/12
- added R5: 100, rcl:R-EU_0309/10
Connections:
- new net +5V: C2.1, IC1.VCC1, R5.2, U$1.+5V
- new net N$17: SDA.1, U$1.A4
- new net N$18: SCL.1, U$1.A5
- new net N$19: ARDUINO_LED.1, U$1.D13
- new net N$20: U$1.D12, WHISKER.1
- new net N$21: BUTTON.1, U$1.D11
- new net N$22: NEOPIXEL.1, U$1.D7
- new net N$23: IR1.OUT, U$1.D4
- new net N$24: R4.1, U$1.D5
- new net VCC: C4.+, C5.1, IR1.VCC, R5.1
- net GND: now also C4.-, C5.2, IR-LED.C, IR1.GND
- net N$12: now also IR-LED.A, R4.2; no longer C2.1, IC1.VCC1, U$1.+5V
Other:
- moved on the sheet: LEFTLED, R1, R2, RIGHTLED

Commit message: bluetooth modul hc05 connection added
Parts:
- added BLUETOOTH_HC05: (no value), pinhead:PINHD-1X6
Connections:
- new net BLUE_KEY: BLUETOOTH_HC05.5
- new net BLUE_LED: BLUETOOTH_HC05.6
- new net BLUE_RXD_ARDUINO_TXD: BLUETOOTH_HC05.4, U$1.D8
- new net BLUE_TXD_ARDUINO_RXD: BLUETOOTH_HC05.3, U$1.D6
- net +5V: now also BLUETOOTH_HC05.1
- net GND: now also BLUETOOTH_HC05.2
Other:
- moved on the sheet: NEOPIXEL
Changed lines of the file:
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@@
 <part name="C5" library="rcl" deviceset="C-EU" device="050-025X075" value="100n"/>
 <part name="R5" library="rcl" deviceset="R-EU_" device="0309/10" value="100"/>
+<part name="BLUETOOTH_HC05" library="pinhead" deviceset="PINHD-1X6" device=""/>
+<part name="GND13" library="supply1" deviceset="GND" device=""/>
+<part name="SUPPLY3" library="supply2" deviceset="+5V" device=""/>
 </parts>
 <sheets>
@@
 <instance part="SDA" gate="G$1" x="111.76" y="68.58" rot="R90"/>
 <instance part="SCL" gate="G$1" x="106.68" y="78.74" rot="R90"/>
-<instance part="NEOPIXEL" gate="G$1" x="121.92" y="17.78" rot="R270"/>
+<instance part="NEOPIXEL" gate="G$1" x="121.92" y="12.7" rot="R270"/>
 <instance part="BUTTON" gate="G$1" x="142.24" y="17.78" rot="R270"/>
 <instance part="WHISKER" gate="G$1" x="147.32" y="7.62" rot="R270"/>
@@
 <instance part="C5" gate="G$1" x="218.44" y="2.54"/>
 <instance part="R5" gate="G$1" x="193.04" y="12.7" rot="R90"/>
+<instance part="BLUETOOTH_HC05" gate="A" x="233.68" y="96.52"/>
+<instance part="GND13" gate="1" x="185.42" y="99.06"/>
+<instance part="SUPPLY3" gate="+5V" x="195.58" y="116.84"/>
 </instances>
 <busses>
@@
 <pinref part="GND12" gate="1" pin="GND"/>
 <wire x1="111.76" y1="-30.48" x2="111.76" y2="-33.02" width="0.1524" layer="91"/>
+</segment>
+<segment>
+<pinref part="BLUETOOTH_HC05" gate="A" pin="2"/>
+<label x="200.66" y="101.6" size="1.778" layer="95"/>
+<pinref part="GND13" gate="1" pin="GND"/>
+<wire x1="231.14" y1="101.6" x2="185.42" y2="101.6" width="0.1524" layer="91"/>
 </segment>
 </net>
@@
 <pinref part="NEOPIXEL" gate="G$1" pin="1"/>
 <pinref part="U$1" gate="G$1" pin="D7"/>
-<wire x1="121.92" y1="20.32" x2="121.92" y2="30.48" width="0.1524" layer="91"/>
+<wire x1="121.92" y1="15.24" x2="121.92" y2="30.48" width="0.1524" layer="91"/>
 </segment>
 </net>
@@
 <pinref part="R5" gate="G$1" pin="2"/>
 </segment>
+<segment>
+<pinref part="SUPPLY3" gate="+5V" pin="+5V"/>
+<wire x1="195.58" y1="114.3" x2="195.58" y2="104.14" width="0.1524" layer="91"/>
+<pinref part="BLUETOOTH_HC05" gate="A" pin="1"/>
+<wire x1="231.14" y1="104.14" x2="195.58" y2="104.14" width="0.1524" layer="91"/>
+<label x="200.66" y="104.14" size="1.778" layer="95"/>
+</segment>
 </net>
 <net name="VCC" class="0">
@@
 </segment>
 </net>
+<net name="BLUE_KEY" class="0">
+<segment>
+<pinref part="BLUETOOTH_HC05" gate="A" pin="5"/>
+<wire x1="231.14" y1="93.98" x2="200.66" y2="93.98" width="0.1524" layer="91"/>
+<label x="195.58" y="93.98" size="1.778" layer="95"/>
+</segment>
+</net>
+<net name="BLUE_LED" class="0">
+<segment>
+<pinref part="BLUETOOTH_HC05" gate="A" pin="6"/>
+<wire x1="231.14" y1="91.44" x2="200.66" y2="91.44" width="0.1524" layer="91"/>
+<label x="195.58" y="91.44" size="1.778" layer="95"/>
+</segment>
+</net>
+<net name="BLUE_TXD_ARDUINO_RXD" class="0">
+<segment>
+<pinref part="BLUETOOTH_HC05" gate="A" pin="3"/>
+<wire x1="231.14" y1="99.06" x2="200.66" y2="99.06" width="0.1524" layer="91"/>
+<label x="195.58" y="99.06" size="1.778" layer="95"/>
+</segment>
+<segment>
+<pinref part="U$1" gate="G$1" pin="D6"/>
+<wire x1="116.84" y1="30.48" x2="116.84" y2="20.32" width="0.1524" layer="91"/>
+<label x="116.84" y="33.02" size="1.778" layer="95" rot="R270"/>
+</segment>
+</net>
+<net name="BLUE_RXD_ARDUINO_TXD" class="0">
+<segment>
+<pinref part="BLUETOOTH_HC05" gate="A" pin="4"/>
+<wire x1="231.14" y1="96.52" x2="200.66" y2="96.52" width="0.1524" layer="91"/>
+<label x="195.58" y="96.52" size="1.778" layer="95"/>
+</segment>
+<segment>
+<pinref part="U$1" gate="G$1" pin="D8"/>
+<wire x1="127" y1="30.48" x2="127" y2="20.32" width="0.1524" layer="91"/>
+<label x="127" y="33.02" size="1.778" layer="95" rot="R270"/>
+</segment>
+</net>

Commit message: additional pins in schematic added
Parts:
- added 3V3, A6, A7, AREF, RESET, RX, TX: (no value), pinhead:PINHD-1X1
- added A1: V5V, pinhead:PINHD-1X1
- added A2: VGND, pinhead:PINHD-1X1
Connections:
- new net N$25: A6.1, U$1.A6
- new net N$26: 3V3.1, U$1.3V3
- new net N$27: AREF.1, U$1.AREF
- new net N$28: A7.1, U$1.A7
- new net N$29: RESET.1, U$1.RESET
- new net N$30: TX.1, U$1.D1/TX
- new net N$31: RX.1, U$1.D0/RX
- net +5V: now also A1.1
- net GND: now also A2.1
Other:
- moved on the sheet: BUTTON, WHISKER
Changed lines of the file:
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@@
 <part name="GND13" library="supply1" deviceset="GND" device=""/>
 <part name="SUPPLY3" library="supply2" deviceset="+5V" device=""/>
+<part name="A7" library="pinhead" deviceset="PINHD-1X1" device=""/>
+<part name="AREF" library="pinhead" deviceset="PINHD-1X1" device=""/>
+<part name="TX" library="pinhead" deviceset="PINHD-1X1" device=""/>
+<part name="A6" library="pinhead" deviceset="PINHD-1X1" device=""/>
+<part name="3V3" library="pinhead" deviceset="PINHD-1X1" device=""/>
+<part name="RX" library="pinhead" deviceset="PINHD-1X1" device=""/>
+<part name="RESET" library="pinhead" deviceset="PINHD-1X1" device=""/>
+<part name="A1" library="pinhead" deviceset="PINHD-1X1" device="" value="V5V"/>
+<part name="A2" library="pinhead" deviceset="PINHD-1X1" device="" value="VGND"/>
+<part name="SUPPLY4" library="supply2" deviceset="+5V" device=""/>
+<part name="GND14" library="supply1" deviceset="GND" device=""/>
 </parts>
 <sheets>
@@
 <instance part="SDA" gate="G$1" x="111.76" y="68.58" rot="R90"/>
 <instance part="SCL" gate="G$1" x="106.68" y="78.74" rot="R90"/>
-<instance part="NEOPIXEL" gate="G$1" x="121.92" y="12.7" rot="R270"/>
-<instance part="BUTTON" gate="G$1" x="142.24" y="17.78" rot="R270"/>
-<instance part="WHISKER" gate="G$1" x="147.32" y="7.62" rot="R270"/>
+<instance part="NEOPIXEL" gate="G$1" x="121.92" y="12.7" smashed="yes" rot="R270">
+<attribute name="NAME" x="122.555" y="31.75" size="1.778" layer="95" rot="R270"/>
+<attribute name="VALUE" x="116.84" y="19.05" size="1.778" layer="96" rot="R270"/>
+</instance>
+<instance part="BUTTON" gate="G$1" x="142.24" y="22.86" rot="R270"/>
+<instance part="WHISKER" gate="G$1" x="147.32" y="10.16" rot="R270"/>
 <instance part="IR1" gate="G$1" x="193.04" y="-7.62" rot="MR0"/>
 <instance part="GND9" gate="1" x="193.04" y="-27.94"/>
@@
 <instance part="GND13" gate="1" x="185.42" y="99.06"/>
 <instance part="SUPPLY3" gate="+5V" x="195.58" y="116.84"/>
+<instance part="A7" gate="G$1" x="96.52" y="78.74" rot="R90"/>
+<instance part="AREF" gate="G$1" x="137.16" y="78.74" rot="R90"/>
+<instance part="TX" gate="G$1" x="76.2" y="12.7" rot="R270"/>
+<instance part="A6" gate="G$1" x="101.6" y="68.58" rot="R90"/>
+<instance part="3V3" gate="G$1" x="142.24" y="68.58" rot="R90"/>
+<instance part="RX" gate="G$1" x="81.28" y="22.86" rot="R270"/>
+<instance part="RESET" gate="G$1" x="86.36" y="17.78" rot="R270"/>
+<instance part="A1" gate="G$1" x="233.68" y="58.42" rot="R270"/>
+<instance part="A2" gate="G$1" x="233.68" y="45.72" rot="R90"/>
+<instance part="SUPPLY4" gate="+5V" x="233.68" y="71.12"/>
+<instance part="GND14" gate="1" x="233.68" y="33.02"/>
 </instances>
 <busses>
@@
 <pinref part="GND13" gate="1" pin="GND"/>
 <wire x1="231.14" y1="101.6" x2="185.42" y2="101.6" width="0.1524" layer="91"/>
+</segment>
+<segment>
+<pinref part="GND14" gate="1" pin="GND"/>
+<pinref part="A2" gate="G$1" pin="1"/>
+<wire x1="233.68" y1="35.56" x2="233.68" y2="43.18" width="0.1524" layer="91"/>
 </segment>
 </net>
@@
 <pinref part="WHISKER" gate="G$1" pin="1"/>
 <pinref part="U$1" gate="G$1" pin="D12"/>
-<wire x1="147.32" y1="10.16" x2="147.32" y2="30.48" width="0.1524" layer="91"/>
+<wire x1="147.32" y1="12.7" x2="147.32" y2="30.48" width="0.1524" layer="91"/>
 </segment>
 </net>
@@
 <pinref part="BUTTON" gate="G$1" pin="1"/>
 <pinref part="U$1" gate="G$1" pin="D11"/>
-<wire x1="142.24" y1="20.32" x2="142.24" y2="30.48" width="0.1524" layer="91"/>
+<wire x1="142.24" y1="25.4" x2="142.24" y2="30.48" width="0.1524" layer="91"/>
 </segment>
 </net>
@@
 <label x="200.66" y="104.14" size="1.778" layer="95"/>
 </segment>
+<segment>
+<pinref part="SUPPLY4" gate="+5V" pin="+5V"/>
+<pinref part="A1" gate="G$1" pin="1"/>
+<wire x1="233.68" y1="68.58" x2="233.68" y2="60.96" width="0.1524" layer="91"/>
+</segment>
 </net>
 <net name="VCC" class="0">
@@
 <pinref part="U$1" gate="G$1" pin="D6"/>
 <wire x1="116.84" y1="30.48" x2="116.84" y2="20.32" width="0.1524" layer="91"/>
-<label x="116.84" y="33.02" size="1.778" layer="95" rot="R270"/>
+<label x="116.84" y="20.32" size="1.778" layer="95" rot="R270"/>
 </segment>
 </net>
@@
 <pinref part="U$1" gate="G$1" pin="D8"/>
 <wire x1="127" y1="30.48" x2="127" y2="20.32" width="0.1524" layer="91"/>
-<label x="127" y="33.02" size="1.778" layer="95" rot="R270"/>
-</segment>
-</net>
+<label x="127" y="20.32" size="1.778" layer="95" rot="R270"/>
+</segment>
+</net>
+<net name="N$25" class="0">
+<segment>
+<pinref part="U$1" gate="G$1" pin="A6"/>
+<pinref part="A6" gate="G$1" pin="1"/>
+<wire x1="101.6" y1="66.04" x2="101.6" y2="60.96" width="0.1524" layer="91"/>
+</segment>
+</net>
+<net name="N$26" class="0">
+<segment>
+<pinref part="U$1" gate="G$1" pin="3V3"/>
+<pinref part="3V3" gate="G$1" pin="1"/>
+<wire x1="142.24" y1="66.04" x2="142.24" y2="60.96" width="0.1524" layer="91"/>
+</segment>
+</net>
+<net name="N$27" class="0">
+<segment>
+<pinref part="U$1" gate="G$1" pin="AREF"/>
+<pinref part="AREF" gate="G$1" pin="1"/>
+<wire x1="137.16" y1="60.96" x2="137.16" y2="76.2" width="0.1524" layer="91"/>
+</segment>
+</net>
+<net name="N$28" class="0">
+<segment>
+<pinref part="U$1" gate="G$1" pin="A7"/>
+<pinref part="A7" gate="G$1" pin="1"/>
+<wire x1="96.52" y1="60.96" x2="96.52" y2="76.2" width="0.1524" layer="91"/>
+</segment>
+</net>
+<net name="N$30" class="0">
+<segment>
+<pinref part="TX" gate="G$1" pin="1"/>
+<pinref part="U$1" gate="G$1" pin="D1/TX"/>
+<wire x1="76.2" y1="15.24" x2="76.2" y2="30.48" width="0.1524" layer="91"/>
+</segment>
+</net>
+<net name="N$31" class="0">
+<segment>
+<pinref part="RX" gate="G$1" pin="1"/>
+<pinref part="U$1" gate="G$1" pin="D0/RX"/>
+<wire x1="81.28" y1="25.4" x2="81.28" y2="30.48" width="0.1524" layer="91"/>
+</segment>
+</net>
+<net name="N$29" class="0">
+<segment>
+<pinref part="RESET" gate="G$1" pin="1"/>
+<pinref part="U$1" gate="G$1" pin="RESET"/>
+<wire x1="86.36" y1="20.32" x2="86.36" y2="30.48" width="0.1524" layer="91"/>
+</segment>
+</net>
